File: wifi-50A-relay.kicad_pcb (KiCad board)
At the start: 2 copper layers, 85 x 56 mm, 40 parts, among them J1 PROG, J2 100k_HOT, J3 100k_COLD, K1 J115F21C12VDCS.9, K2 J115F21C12VDCS.9, Q1 AO3400A, SW1 SKRKAEE020, U1 ESP-WROOM-02, U2 TPS54331DR, U3 ADS1115IDGS

Commit message: Fix programming error
Connections:
- D3 pad 4: Net-(D3-Pad4) -> unconnected-(D3-Pad4)
- K1 pad 12: Net-(K1-Pad12) -> unconnected-(K1-Pad12)
- K1 pad 14: Net-(K1-Pad14) -> unconnected-(K1-Pad14)
- K2 pad 12: Net-(K2-Pad12) -> unconnected-(K2-Pad12)
- K2 pad 14: Net-(K2-Pad14) -> unconnected-(K2-Pad14)
- U1 pad 14: Net-(U1-Pad14) -> unconnected-(U1-Pad14)
- U1 pad 15: Net-(U1-Pad15) -> unconnected-(U1-Pad15)
- U1 pad 16: Net-(U1-Pad16) -> unconnected-(U1-Pad16)
- U1 pad 17: Net-(U1-Pad17) -> unconnected-(U1-Pad17)
- U1 pad 4: Net-(U1-Pad4) -> unconnected-(U1-Pad4)
- U1 pad 5: Net-(U1-Pad5) -> unconnected-(U1-Pad5)
- U1 pad 6: Net-(U1-Pad6) -> GND
- U2 pad 3: Net-(U2-Pad3) -> unconnected-(U2-Pad3)
- U3 pad 2: Net-(U3-Pad2) -> unconnected-(U3-Pad2)
Routing:
- net GND: track 40.7 -> 41.9 mm
Other:
- net class Default removed
- net class Mains removed
