File: wifi-50A-relay.kicad_pcb (KiCad board)
At the start: 2 copper layers, 85 x 56 mm, 40 parts, among them J1 PROG, J2 100k_HOT, J3 100k_COLD, K1 J115F21C12VDCS.9, K2 J115F21C12VDCS.9, Q1 AO3400A, SW1 SKRKAEE020, U1 ESP-WROOM-02, U2 TPS54331DR, U3 ADS1115IDGS

Commit message: Add i2c pull-ups
Forgotten in previous revisions
Parts:
- added R13: 10k, Resistor_SMD:R_0402_1005Metric, F.Cu at (95.8, 62.2)
- added R14: 10k, Resistor_SMD:R_0402_1005Metric, F.Cu at (95.8, 63.2)
Routing:
- net +3V3: track 83.7 -> 88.2 mm
- net /SDA: track 27.4 -> 29.8 mm, vias 2 -> 4
- net /SCL: track 33.0 -> 33.5 mm

Commit message: Add more clearance
This is unnessecary, but double the clearance between the mains &
low-voltage side to 8mm since we have the room for it.
Routing:
- net GND: track 41.9 -> 36.0 mm
- net +12V: track 114.4 -> 117.4 mm, vias 0 -> 1
Changed lines of the file:
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@@
     )
     (pad_to_mask_clearance 0)
+    (grid_origin 65.7 61.5)
     (pcbplotparams
       (layerselection 0x00010fc_ffffffff)
@@
     (fp_arc (start 27.84 11.94) (mid 27.617401 12.477401) (end 27.08 12.7) (layer "F.Fab") (width 0.1))
     (pad "11" thru_hole circle locked (at 15.2 -8.9) (size 4 4) (drill 2.1) (layers *.Cu *.Mask)
-      (net 10 "/AC_PH_2") (pintype "passive") (clearance 3.5))
+      (net 10 "/AC_PH_2") (pintype "passive"))
     (pad "12" thru_hole circle locked (at 25.34 8.9) (size 4 4) (drill 2.1) (layers *.Cu *.Mask)
-      (net 19 "unconnected-(K2-Pad12)") (pintype "passive+no_connect") (clearance 3.5))
+      (net 19 "unconnected-(K2-Pad12)") (pintype "passive+no_connect"))
     (pad "14" thru_hole circle locked (at 17.74 8.9) (size 4 4) (drill 2.1) (layers *.Cu *.Mask)
-      (net 20 "unconnected-(K2-Pad14)") (pintype "passive+no_connect") (clearance 3.5))
+      (net 20 "unconnected-(K2-Pad14)") (pintype "passive+no_connect"))
     (pad "A1" thru_hole roundrect locked (at 2.54 -5.1) (size 2 2) (drill 1.1) (layers *.Cu *.Mask) (roundrect_rratio 0.25)
       (net 2 "+12V") (pintype "passive"))
@@
   (gr_arc (start 113 84) (mid 112.12132 86.12132) (end 110 87) (layer "Edge.Cuts") (width 0.05))
   (gr_line (start 53 39) (end 70 39) (layer "Edge.Cuts") (width 0.05))
-  (segment (start 79.269999 43.730001) (end 79.539998 44) (width 3) (layer "F.Cu") (net 1))
-  (segment (start 82 44) (end 82 44) (width 3) (layer "F.Cu") (net 1))
-  (segment (start 84 44) (end 87 44) (width 3) (layer "F.Cu") (net 1))
   (segment (start 92.7625 46) (end 92 46) (width 0.25) (layer "F.Cu") (net 1))
-  (segment (start 82 44) (end 84 44) (width 3) (layer "F.Cu") (net 1))
-  (segment (start 51 44) (end 52.300011 42.699989) (width 3) (layer "F.Cu") (net 1))
   (segment (start 100.43 72.8) (end 100.43 73.67) (width 0.127) (layer "F.Cu") (net 1))
+  (segment (start 79.269999 43.730001) (end 81.730001 43.730001) (width 1) (layer "F.Cu") (net 1))
   (segment (start 100.43 71.92) (end 100.45 71.9) (width 0.127) (layer "F.Cu") (net 1))
-  (segment (start 79.539998 44) (end 82 44) (width 3) (layer "F.Cu") (net 1))
   (segment (start 92 46) (end 91.75 45.75) (width 0.25) (layer "F.Cu") (net 1))
+  (segment (start 81.730001 43.730001) (end 82 44) (width 1) (layer "F.Cu") (net 1))
   (segment (start 100.43 73.67) (end 100.4 73.7) (width 0.127) (layer "F.Cu") (net 1))
   (segment (start 100.43 72.8) (end 100.43 71.92) (width 0.127) (layer "F.Cu") (net 1))
-  (segment (start 63.114512 42.699989) (end 78.239987 42.699989) (width 3) (layer "F.Cu") (net 1))
-  (segment (start 78.239987 42.699989) (end 79.269999 43.730001) (width 3) (layer "F.Cu") (net 1))
-  (segment (start 52.300011 42.699989) (end 63.114512 42.699989) (width 3) (layer "F.Cu") (net 1))
   (via (at 100.9 68.1) (size 0.6) (drill 0.3) (layers "F.Cu" "B.Cu") (net 1))
   (via (at 87 55.4) (size 0.6) (drill 0.3) (layers "F.Cu" "B.Cu") (net 1))
@@
   (via (at 106.7 58) (size 0.6) (drill 0.3) (layers "F.Cu" "B.Cu") (net 1))
   (segment (start 100.4 74.7) (end 100.5 74.8) (width 0.25) (layer "B.Cu") (net 1))
+  (segment (start 51 44) (end 79 44) (width 1) (layer "B.Cu") (net 1))
+  (segment (start 79 44) (end 79.269999 43.730001) (width 1) (layer "B.Cu") (net 1))
   (segment (start 100.4 73) (end 100.4 74.7) (width 0.25) (layer "B.Cu") (net 1))
-  (segment (start 52.799999 47.200001) (end 46.200001 47.200001) (width 3) (layer "F.Cu") (net 2))
-  (segment (start 79.125 75.875) (end 77.5 74.25) (width 0.25) (layer "F.Cu") (net 2))
-  (segment (start 77.5 49.25) (end 74.149999 45.899999) (width 3) (layer "F.Cu") (net 2))
-  (segment (start 80.35 77.1) (end 79.125 75.875) (width 0.25) (layer "F.Cu") (net 2))
   (segment (start 106.35 71.3) (end 106.35 70.35) (width 0.25) (layer "F.Cu") (net 2))
   (segment (start 103.21001 72.51001) (end 105.86499 72.51001) (width 0.5) (layer "F.Cu") (net 2))
-  (segment (start 77.65 49.1) (end 77.5 49.25) (width 0.25) (layer "F.Cu") (net 2))
   (segment (start 106.35 72.025) (end 106.35 71.3) (width 0.5) (layer "F.Cu") (net 2))
   (segment (start 99.6 68.9) (end 103.21001 72.51001) (width 0.5) (layer "F.Cu") (net 2))
-  (segment (start 74.149999 45.899999) (end 54.100001 45.899999) (width 3) (layer "F.Cu") (net 2))
-  (segment (start 77.5 69.1) (end 80.7 69.1) (width 0.5) (layer "F.Cu") (net 2))
   (segment (start 106.465 68.975) (end 106.465 70.235) (width 0.25) (layer "F.Cu") (net 2))
-  (segment (start 80.46 49.1) (end 77.65 49.1) (width 0.25) (layer "F.Cu") (net 2))
-  (segment (start 77.5 69.1) (end 77.5 74.25) (width 3) (layer "F.Cu") (net 2))
   (segment (start 80.9 68.9) (end 99.6 68.9) (width 0.5) (layer "F.Cu") (net 2))
   (segment (start 106.35 70.35) (end 106.465 70.235) (width 0.25) (layer "F.Cu") (net 2))
@@
   (segment (start 80.7 69.1) (end 80.9 68.9) (width 0.5) (layer "F.Cu") (net 2))
   (segment (start 80.46 77.1) (end 80.35 77.1) (width 0.25) (layer "F.Cu") (net 2))
-  (segment (start 77.5 49.25) (end 77.5 69.1) (width 3) (layer "F.Cu") (net 2))
   (segment (start 84.6 49.1) (end 89.25 53.75) (width 0.25) (layer "F.Cu") (net 2))
-  (segment (start 54.100001 45.899999) (end 52.799999 47.200001) (width 3) (layer "F.Cu") (net 2))
-  (segment (start 46.200001 47.200001) (end 43 44) (width 3) (layer "F.Cu") (net 2))
   (segment (start 105.86499 72.51001) (end 106.35 72.025) (width 0.5) (layer "F.Cu") (net 2))
+  (via (at 80.9 68.9) (size 0.6) (drill 0.3) (layers "F.Cu" "B.Cu") (net 2))
+  (segment (start 77.89952 45.19952) (end 77.89952 46.44952) (width 1) (layer "B.Cu") (net 2))
+  (segment (start 52.200009 46.199511) (end 53.2 45.19952) (width 1) (layer "B.Cu") (net 2))
+  (segment (start 77.89952 69.05048) (end 77.89952 74.69952) (width 1) (layer "B.Cu") (net 2))
+  (segment (start 45.199511 46.199511) (end 52.200009 46.199511) (width 1) (layer "B.Cu") (net 2))
+  (segment (start 53.2 45.19952) (end 77.89952 45.19952) (width 1) (layer "B.Cu") (net 2))
+  (segment (start 77.949511 69.000489) (end 80.799511 69.000489) (width 1) (layer "B.Cu") (net 2))
+  (segment (start 43 44) (end 45.199511 46.199511) (width 1) (layer "B.Cu") (net 2))
+  (segment (start 80.799511 69.000489) (end 80.9 68.9) (width 1) (layer "B.Cu") (net 2))
+  (segment (start 77.89952 46.44952) (end 77.89952 69.05048) (width 1) (layer "B.Cu") (net 2))
+  (segment (start 77.89952 74.69952) (end 80.45 77.25) (width 1) (layer "B.Cu") (net 2))
+  (segment (start 77.89952 46.44952) (end 80.45 49) (width 1) (layer "B.Cu") (net 2))
+  (segment (start 77.89952 69.05048) (end 77.949511 69.000489) (width 1) (layer "B.Cu") (net 2))
   (segment (start 110.7 69.125) (end 109.225 69.125) (width 0.127) (layer "F.Cu") (net 3))
   (segment (start 109.225 69.125) (end 109 68.9) (width 0.127) (layer "F.Cu") (net 3))
