File: wifi-30A-relay.kicad_pcb (KiCad board)
At the start: 2 copper layers, 85 x 56 mm, 42 parts, among them J1 PROG, K1 J115F21C12VDCS.9, K2 J115F21C12VDCS.9, Q1 AO3400A, SW1 SKRKAEE020, U1 ESP-WROOM-02, U2 TPS54331DR, U3 ADS1115IDGS

Commit message: Add readme & license, rename files
Parts:
- K1, K2: footprint wifi-50A-relay:Relay_SPDT_CIT-J115F2 -> wifi-30A-relay:Relay_SPDT_CIT-J115F2
Other:
- board text added: "30A water heater controller flaviutamas.com/p/50a-wh-controller"
- board text removed: "50A water heater controller flaviutamas.com/p/50a-wh-controller"
