File: wifi-30A-relay.kicad_sch (KiCad schematic)
At the start: 42 parts, among them J1 PROG, J2 100k_HOT, J3 100k_COLD, K1 J115F21C12VDCS.9, K2 J115F21C12VDCS.9, Q1 AO3400A, SW1 SKRKAEE020, U1 ESP-WROOM-02, U2 TPS54331DR, U3 ADS1115IDGS

Commit message: Add readme & license, rename files
Parts:
- K1, K2: footprint wifi-50A-relay:Relay_SPDT_CIT-J115F2 -> wifi-30A-relay:Relay_SPDT_CIT-J115F2
Changed lines of the file:
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@@
       (effects (font (size 1.27 1.27)) (justify left))
     )
-    (property "Footprint" "wifi-50A-relay:Relay_SPDT_CIT-J115F2" (id 2) (at 231.14 48.26 0)
+    (property "Footprint" "wifi-30A-relay:Relay_SPDT_CIT-J115F2" (id 2) (at 231.14 48.26 0)
       (effects (font (size 1.27 1.27)) (justify left) hide)
     )
@@
       (effects (font (size 1.27 1.27)) (justify left))
     )
-    (property "Footprint" "wifi-50A-relay:Relay_SPDT_CIT-J115F2" (id 2) (at 189.23 48.26 0)
+    (property "Footprint" "wifi-30A-relay:Relay_SPDT_CIT-J115F2" (id 2) (at 189.23 48.26 0)
       (effects (font (size 1.27 1.27)) (justify left) hide)
     )
@@
     )
     (path "/00000000-0000-0000-0000-000061161134"
-      (reference "K1") (unit 1) (value "J115F21C12VDCS.9") (footprint "wifi-50A-relay:Relay_SPDT_CIT-J115F2")
+      (reference "K1") (unit 1) (value "J115F21C12VDCS.9") (footprint "wifi-30A-relay:Relay_SPDT_CIT-J115F2")
     )
     (path "/00000000-0000-0000-0000-00006115ee47"
-      (reference "K2") (unit 1) (value "J115F21C12VDCS.9") (footprint "wifi-50A-relay:Relay_SPDT_CIT-J115F2")
+      (reference "K2") (unit 1) (value "J115F21C12VDCS.9") (footprint "wifi-30A-relay:Relay_SPDT_CIT-J115F2")
     )
     (path "/00000000-0000-0000-0000-00006117b67d"
